Commit message: corrected hand to be right handed instead of left handed because I am an idiot sometimes

File: urdf/hand.urdf (robot description, URDF)
Before this commit: robot robot_hand, 21 links, 20 joints
Joints:
- joint base_to_thumb: limit lower=0.0 upper=1.5708 effort=1000.0 velocity=0.5 -> lower=0.0 upper=-1.5708 effort=1000.0 velocity=0.5
- joint fore_finger_inter_to_distal: limit lower=0.0 upper=1.5708 effort=1000.0 velocity=0.5 -> lower=0.0 upper=-1.5708 effort=1000.0 velocity=0.5
- joint fore_finger_meta_to_proximal: limit lower=0.0 upper=1.5708 effort=1000.0 velocity=0.5 -> lower=0.0 upper=-1.5708 effort=1000.0 velocity=0.5
- joint fore_finger_proximal_to_inter: limit lower=0.0 upper=1.5708 effort=1000.0 velocity=0.5 -> lower=0.0 upper=-1.5708 effort=1000.0 velocity=0.5
- joint little_finger_meta_to_proximal: limit lower=0.0 upper=1.5708 effort=1000.0 velocity=0.5 -> lower=0.0 upper=-1.5708 effort=1000.0 velocity=0.5
- joint little_finger_proximal_to_inter: limit lower=0.0 upper=1.5708 effort=1000.0 velocity=0.5 -> lower=0.0 upper=-1.5708 effort=1000.0 velocity=0.5
- joint middle_finger_inter_to_distal: limit lower=0.0 upper=1.5708 effort=1000.0 velocity=0.5 -> lower=0.0 upper=-1.5708 effort=1000.0 velocity=0.5
- joint middle_finger_meta_to_proximal: limit lower=0.0 upper=1.5708 effort=1000.0 velocity=0.5 -> lower=0.0 upper=-1.5708 effort=1000.0 velocity=0.5
- joint middle_finger_proximal_to_inter: limit lower=0.0 upper=1.5708 effort=1000.0 velocity=0.5 -> lower=0.0 upper=-1.5708 effort=1000.0 velocity=0.5
- joint ring_finger_inter_to_distal: limit lower=0.0 upper=1.5708 effort=1000.0 velocity=0.5 -> lower=0.0 upper=-1.5708 effort=1000.0 velocity=0.5
- joint ring_finger_meta_to_proximal: limit lower=0.0 upper=1.5708 effort=1000.0 velocity=0.5 -> lower=0.0 upper=-1.5708 effort=1000.0 velocity=0.5
- joint ring_finger_proximal_to_inter: limit lower=0.0 upper=1.5708 effort=1000.0 velocity=0.5 -> lower=0.0 upper=-1.5708 effort=1000.0 velocity=0.5
- joint thumb_meta_to_distal: limit lower=0.0 upper=1.5708 effort=1000.0 velocity=0.5 -> lower=0.0 upper=-1.5708 effort=1000.0 velocity=0.5
- joint thumb_meta_to_proximal: limit lower=0.0 upper=1.5708 effort=1000.0 velocity=0.5 -> lower=0.0 upper=-1.5708 effort=1000.0 velocity=0.5
- joint thumb_meta_to_proximal_zero: limit lower=0.0 upper=0.3 effort=1000.0 velocity=0.5 -> lower=0.0 upper=-0.3 effort=1000.0 velocity=0.5
